File: hardware/cole-1-caps.sch (KiCad schematic (older format))
At the start: 10 parts

Commit message: Final schematic and PCB layout.
Parts:
- added C11: 0.1u, Capacitors_SMD:C_0805_HandSoldering, symbol C_Small
- C1: footprint Capacitors_THT:C_Disc_D4.7mm_W2.5mm_P5.00mm -> Capacitors_SMD:C_0805_HandSoldering
- C10: renamed from C11; footprint Capacitors_THT:C_Disc_D4.7mm_W2.5mm_P5.00mm -> Capacitors_SMD:C_0805_HandSoldering
- C2: renamed from C3; footprint Capacitors_THT:C_Disc_D4.7mm_W2.5mm_P5.00mm -> Capacitors_SMD:C_0805_HandSoldering
- C3: renamed from C4; footprint Capacitors_THT:C_Disc_D4.7mm_W2.5mm_P5.00mm -> Capacitors_SMD:C_0805_HandSoldering
- C4: renamed from C5; footprint Capacitors_THT:C_Disc_D4.7mm_W2.5mm_P5.00mm -> Capacitors_SMD:C_0805_HandSoldering
- C5: renamed from C6; footprint Capacitors_THT:C_Disc_D4.7mm_W2.5mm_P5.00mm -> Capacitors_SMD:C_0805_HandSoldering
- C6: renamed from C7; footprint Capacitors_THT:C_Disc_D4.7mm_W2.5mm_P5.00mm -> Capacitors_SMD:C_0805_HandSoldering
- C7: renamed from C8; footprint Capacitors_THT:C_Disc_D4.7mm_W2.5mm_P5.00mm -> Capacitors_SMD:C_0805_HandSoldering
- C8: renamed from C9; footprint Capacitors_THT:C_Disc_D4.7mm_W2.5mm_P5.00mm -> Capacitors_SMD:C_0805_HandSoldering
- C9: renamed from C10; footprint Capacitors_THT:C_Disc_D4.7mm_W2.5mm_P5.00mm -> Capacitors_SMD:C_0805_HandSoldering
Connections:
- net GND: now also C11.1
- net VCC: now also C11.2
Changed lines of the file:
@@
 $EndDescr
 $Comp
-L C_Small C6
+L C_Small C5
 U 1 1 5A48259A
 P 5650 4100
-F 0 "C6" V 5500 4050 50  0000 L CNN
+F 0 "C5" V 5500 4050 50  0000 L CNN
 F 1 "0.1u" V 5800 4050 50  0001 L CNN
-F 2 "Capacitors_THT:C_Disc_D4.7mm_W2.5mm_P5.00mm" H 5650 4100 50  0001 C CNN
+F 2 "Capacitors_SMD:C_0805_HandSoldering" H 5650 4100 50  0001 C CNN
 F 3 "" H 5650 4100 50  0001 C CNN
 	1    5650 4100
@@
 $EndComp
 $Comp
-L C_Small C7
+L C_Small C6
 U 1 1 5A4827B9
 P 5650 4400
-F 0 "C7" V 5500 4350 50  0000 L CNN
+F 0 "C6" V 5500 4350 50  0000 L CNN
 F 1 "0.1u" V 5800 4350 50  0001 L CNN
-F 2 "Capacitors_THT:C_Disc_D4.7mm_W2.5mm_P5.00mm" H 5650 4400 50  0001 C CNN
+F 2 "Capacitors_SMD:C_0805_HandSoldering" H 5650 4400 50  0001 C CNN
 F 3 "" H 5650 4400 50  0001 C CNN
 	1    5650 4400
@@
 $EndComp
 $Comp
-L C_Small C8
+L C_Small C7
 U 1 1 5A48281D
 P 5650 4700
-F 0 "C8" V 5500 4650 50  0000 L CNN
+F 0 "C7" V 5500 4650 50  0000 L CNN
 F 1 "0.1u" V 5800 4650 50  0001 L CNN
-F 2 "Capacitors_THT:C_Disc_D4.7mm_W2.5mm_P5.00mm" H 5650 4700 50  0001 C CNN
+F 2 "Capacitors_SMD:C_0805_HandSoldering" H 5650 4700 50  0001 C CNN
 F 3 "" H 5650 4700 50  0001 C CNN
 	1    5650 4700
@@
 $EndComp
 $Comp
-L C_Small C9
+L C_Small C8
 U 1 1 5A482823
 P 5650 5000
-F 0 "C9" V 5500 4950 50  0000 L CNN
+F 0 "C8" V 5500 4950 50  0000 L CNN
 F 1 "0.1u" V 5800 4950 50  0001 L CNN
-F 2 "Capacitors_THT:C_Disc_D4.7mm_W2.5mm_P5.00mm" H 5650 5000 50  0001 C CNN
+F 2 "Capacitors_SMD:C_0805_HandSoldering" H 5650 5000 50  0001 C CNN
 F 3 "" H 5650 5000 50  0001 C CNN
 	1    5650 5000
@@
 F 0 "C1" V 5500 2850 50  0000 L CNN
 F 1 "0.1u" V 5800 2850 50  0001 L CNN
-F 2 "Capacitors_THT:C_Disc_D4.7mm_W2.5mm_P5.00mm" H 5650 2900 50  0001 C CNN
+F 2 "Capacitors_SMD:C_0805_HandSoldering" H 5650 2900 50  0001 C CNN
 F 3 "" H 5650 2900 50  0001 C CNN
 	1    5650 2900
@@
 $EndComp
 $Comp
-L C_Small C3
+L C_Small C2
 U 1 1 5A4829A3
 P 5650 3200
-F 0 "C3" V 5500 3150 50  0000 L CNN
+F 0 "C2" V 5500 3150 50  0000 L CNN
 F 1 "0.1u" V 5800 3150 50  0001 L CNN
-F 2 "Capacitors_THT:C_Disc_D4.7mm_W2.5mm_P5.00mm" H 5650 3200 50  0001 C CNN
+F 2 "Capacitors_SMD:C_0805_HandSoldering" H 5650 3200 50  0001 C CNN
 F 3 "" H 5650 3200 50  0001 C CNN
 	1    5650 3200
@@
 $EndComp
 $Comp
-L C_Small C4
+L C_Small C3
 U 1 1 5A4829A9
 P 5650 3500
-F 0 "C4" V 5500 3450 50  0000 L CNN
+F 0 "C3" V 5500 3450 50  0000 L CNN
 F 1 "0.1u" V 5800 3450 50  0001 L CNN
-F 2 "Capacitors_THT:C_Disc_D4.7mm_W2.5mm_P5.00mm" H 5650 3500 50  0001 C CNN
+F 2 "Capacitors_SMD:C_0805_HandSoldering" H 5650 3500 50  0001 C CNN
 F 3 "" H 5650 3500 50  0001 C CNN
 	1    5650 3500
@@
 $EndComp
 $Comp
-L C_Small C5
+L C_Small C4
 U 1 1 5A4829AF
 P 5650 3800
-F 0 "C5" V 5500 3750 50  0000 L CNN
+F 0 "C4" V 5500 3750 50  0000 L CNN
 F 1 "0.1u" V 5800 3750 50  0001 L CNN
-F 2 "Capacitors_THT:C_Disc_D4.7mm_W2.5mm_P5.00mm" H 5650 3800 50  0001 C CNN
+F 2 "Capacitors_SMD:C_0805_HandSoldering" H 5650 3800 50  0001 C CNN
 F 3 "" H 5650 3800 50  0001 C CNN
 	1    5650 3800
@@
 $EndComp
 $Comp
-L C_Small C10
+L C_Small C9
 U 1 1 5A4829D5
 P 5650 5300
-F 0 "C10" V 5500 5250 50  0000 L CNN
+F 0 "C9" V 5500 5250 50  0000 L CNN
 F 1 "0.1u" V 5800 5250 50  0001 L CNN
-F 2 "Capacitors_THT:C_Disc_D4.7mm_W2.5mm_P5.00mm" H 5650 5300 50  0001 C CNN
+F 2 "Capacitors_SMD:C_0805_HandSoldering" H 5650 5300 50  0001 C CNN
 F 3 "" H 5650 5300 50  0001 C CNN
 	1    5650 5300
@@
 $EndComp
 $Comp
-L GND #PWR019
+L GND #PWR020
 U 1 1 5A482A89
-P 5950 5850
-F 0 "#PWR019" H 5950 5600 50  0001 C CNN
-F 1 "GND" H 5950 5700 50  0000 C CNN
-F 2 "" H 5950 5850 50  0001 C CNN
-F 3 "" H 5950 5850 50  0001 C CNN
-	1    5950 5850
+P 5950 6350
+F 0 "#PWR020" H 5950 6100 50  0001 C CNN
+F 1 "GND" H 5950 6200 50  0000 C CNN
+F 2 "" H 5950 6350 50  0001 C CNN
+F 3 "" H 5950 6350 50  0001 C CNN
+	1    5950 6350
 	1    0    0    -1
 $EndComp
 Wire Wire Line
-	5950 2900 5950 5850
+	5950 2900 5950 6350
 Wire Wire Line
 	5950 2900 5750 2900
@@
 	5550 2900 5350 2900
 $Comp
-L VCC #PWR020
+L VCC #PWR021
 U 1 1 5A482C0A
 P 5350 2550
-F 0 "#PWR020" H 5350 2400 50  0001 C CNN
+F 0 "#PWR021" H 5350 2400 50  0001 C CNN
 F 1 "VCC" H 5350 2700 50  0000 C CNN
 F 2 "" H 5350 2550 50  0001 C CNN
@@
 $EndComp
 Wire Wire Line
-	5350 2550 5350 5600
+	5350 2550 5350 5900
 Wire Wire Line
 	5350 5300 5550 5300
@@
 Connection ~ 5350 4400
 $Comp
-L C_Small C11
+L C_Small C10
 U 1 1 5A479889
 P 5650 5600
-F 0 "C11" V 5500 5550 50  0000 L CNN
+F 0 "C10" V 5500 5550 50  0000 L CNN
 F 1 "0.1u" V 5800 5550 50  0001 L CNN
-F 2 "Capacitors_THT:C_Disc_D4.7mm_W2.5mm_P5.00mm" H 5650 5600 50  0001 C CNN
+F 2 "Capacitors_SMD:C_0805_HandSoldering" H 5650 5600 50  0001 C CNN
 F 3 "" H 5650 5600 50  0001 C CNN
 	1    5650 5600
@@
 Connection ~ 5350 5300
 Connection ~ 5950 5600
+$Comp
+L C_Small C11
+U 1 1 5A5A8AB4
+P 5650 5900
+F 0 "C11" V 5500 5850 50  0000 L CNN
+F 1 "0.1u" V 5800 5850 50  0001 L CNN
+F 2 "Capacitors_SMD:C_0805_HandSoldering" H 5650 5900 50  0001 C CNN
+F 3 "" H 5650 5900 50  0001 C CNN
+	1    5650 5900
+	0    1    1    0
+$EndComp
+Wire Wire Line
+	5350 5900 5550 5900
+Wire Wire Line
+	5750 5900 5950 5900
+Connection ~ 5950 5900
+Connection ~ 5350 5600
 $EndSCHEMATC

Commit message: Updated schematics, board layout, and GAL code for COLE-1+
Parts:
- removed C10, C11, C9: 0.1u, Capacitors_SMD:C_0805_HandSoldering, symbol C_Small
- added C1: 470uf, Capacitor_THT:CP_Radial_D13.0mm_P7.50mm, symbol Device:CP
- added H1, H2, H3, H4: MountingHole_Pad, MountingHole:MountingHole_2.5mm_Pad_Via, symbol Mechanical:MountingHole_Pad
- added J1: PORT A, Connector_PinHeader_2.54mm:PinHeader_1x12_P2.54mm_Vertical, symbol cole-1-rescue:Conn_01x12
- added J2: PORT B, Connector_PinHeader_2.54mm:PinHeader_1x12_P2.54mm_Vertical, symbol cole-1-rescue:Conn_01x12
- added J3: TTL Serial, Connector_PinHeader_2.54mm:PinHeader_1x06_P2.54mm_Vertical, symbol cole-1-rescue:Conn_01x06
- C2: renamed from C1; footprint Capacitors_SMD:C_0805_HandSoldering -> Capacitor_SMD:C_0805_2012Metric_Pad1.15x1.40mm_HandSolder; symbol C_Small -> cole-1-rescue:C_Small
- C3: renamed from C2; footprint Capacitors_SMD:C_0805_HandSoldering -> Capacitor_SMD:C_0805_2012Metric_Pad1.15x1.40mm_HandSolder; symbol C_Small -> cole-1-rescue:C_Small
- C4: renamed from C3; footprint Capacitors_SMD:C_0805_HandSoldering -> Capacitor_SMD:C_0805_2012Metric_Pad1.15x1.40mm_HandSolder; symbol C_Small -> cole-1-rescue:C_Small
- C5: renamed from C4; footprint Capacitors_SMD:C_0805_HandSoldering -> Capacitor_SMD:C_0805_2012Metric_Pad1.15x1.40mm_HandSolder; symbol C_Small -> cole-1-rescue:C_Small
- C6: renamed from C5; footprint Capacitors_SMD:C_0805_HandSoldering -> Capacitor_SMD:C_0805_2012Metric_Pad1.15x1.40mm_HandSolder; symbol C_Small -> cole-1-rescue:C_Small
- C7: renamed from C6; footprint Capacitors_SMD:C_0805_HandSoldering -> Capacitor_SMD:C_0805_2012Metric_Pad1.15x1.40mm_HandSolder; symbol C_Small -> cole-1-rescue:C_Small
- C8: renamed from C7; footprint Capacitors_SMD:C_0805_HandSoldering -> Capacitor_SMD:C_0805_2012Metric_Pad1.15x1.40mm_HandSolder; symbol C_Small -> cole-1-rescue:C_Small
- C9: renamed from C8; footprint Capacitors_SMD:C_0805_HandSoldering -> Capacitor_SMD:C_0805_2012Metric_Pad1.15x1.40mm_HandSolder; symbol C_Small -> cole-1-rescue:C_Small
Connections:
- net GND: now also C1.2, H1.1, H2.1, H3.1, H4.1, J1.12 (Pin_12), J2.12 (Pin_12), J3.6 (Pin_6)
- net VCC: now also C1.1, J1.1 (Pin_1), J2.1 (Pin_1), J3.4 (Pin_4)
- new net CA1: J1.10 (Pin_10)
- new net CA2: J1.11 (Pin_11)
- new net CB1: J2.10 (Pin_10)
- new net CB2: J2.11 (Pin_11)
- new net CTS: J3.1 (Pin_1)
- new net PA0: J1.2 (Pin_2)
- new net PA1: J1.3 (Pin_3)
- new net PA2: J1.4 (Pin_4)
- new net PA3: J1.5 (Pin_5)
- new net PA4: J1.6 (Pin_6)
- new net PA5: J1.7 (Pin_7)
- new net PA6: J1.8 (Pin_8)
- new net PA7: J1.9 (Pin_9)
- new net PB0: J2.2 (Pin_2)
- new net PB1: J2.3 (Pin_3)
- new net PB2: J2.4 (Pin_4)
- new net PB3: J2.5 (Pin_5)
- new net PB4: J2.6 (Pin_6)
- new net PB5: J2.7 (Pin_7)
- new net PB6: J2.8 (Pin_8)
- new net PB7: J2.9 (Pin_9)
- new net RTS: J3.5 (Pin_5)
- new net RXD: J3.3 (Pin_3)
- new net TXD: J3.2 (Pin_2)
Other:
- moved on the sheet: C2, C3, C4, C5, C6, C7, C8, C9
